Commit message: gazebo part 1 done

File: basic_stick/urdf/sensor_stick.xacro (robot description, xacro)
@@ -11,5 +11,6 @@
   <xacro:property name="mass_camera" value="0.2" />
   <!--Import gazebo elements-->
-  <xacro:include filename="$(find basic_stick)/urdf/basic_stick.gazebo.xacro" />
+  <!-- <xacro:include filename="$(find basic_stick)/urdf/sensor_stick_mono.gazebo.xacro" /> -->
+  <xacro:include filename="$(find basic_stick)/urdf/sensor_stick_depth.gazebo.xacro" />
   <!--Links-->
   <link name="world"/>
@@ -65,5 +66,5 @@
   </link>
   <!-- RGBD camera -->
-  <!-- <link name="camera_link">
+  <link name="camera_link">
   <collision>
     <origin xyz="-0.016 0 0" rpy="0 0 0"/>
@@ -83,5 +84,5 @@
     <inertia ixx="5.8083e-4" ixy="0" ixz="0" iyy="3.0833e-5" iyz="0" izz="5.9083e-4" />
   </inertial>
-  </link> -->
+  </link>
   <!--Joints-->
   <joint name="fixed_base_joint" type="fixed">

File: fusionbot_description/urdf/fusionbot_sensor.urdf.xacro (robot description, xacro)
@@ -2,4 +2,6 @@
 <robot name="fusionbot" xmlns:xacro="http://www.ros.org/wiki/xacro">
   <xacro:include filename="$(find fusionbot_description)/urdf/materials.xacro" />
+  <!-- <xacro:include filename="$(find fusionbot_description)/urdf/fusionbot_2d_lidar.gazebo.xacro" /> -->
+  <xacro:include filename="$(find fusionbot_description)/urdf/fusionbot_3d_lidar.gazebo.xacro" />
   <link name='base_footprint' />
   <link name="base_link">
