Commit message: ongoing : moving stick

File: basic_stick/urdf/moving_stick.xacro (robot description, xacro)
@@ -11,6 +11,7 @@
   <xacro:property name="mass_camera" value="0.2" />
   <!--Import gazebo elements-->
-  <!-- <xacro:include filename="$(find basic_stick)/urdf/sensor_stick_mono.gazebo.xacro" /> -->
-  <xacro:include filename="$(find basic_stick)/urdf/sensor_stick_depth.gazebo.xacro" />
+  <xacro:include filename="$(find basic_stick)/urdf/sensor_stick_mono.gazebo.xacro" />
+  <!-- <xacro:include filename="$(find basic_stick)/urdf/sensor_stick_depth.gazebo.xacro" /> -->
+  <xacro:include filename="$(find basic_stick)/urdf/ros2_control.gazebo.xacro" />
   <!--Links-->
   <link name="world"/>
@@ -97,9 +98,9 @@
     <origin xyz="0 0 ${length1/2+length2/2}" rpy="0 0 -${pi/2}"/>
   </joint>
-  <joint name="tilt_joint" type="revolute">
+  <joint name="tilt_joint" type="fixed">
     <origin xyz="0.05 0 ${length2/2+0.02}" rpy="0 0.5 0" />
     <parent link="link_2" />
     <child link="camera_link" />
-    <axis xyz="0 1 0"/>
+    <!-- <axis xyz="0 1 0"/> -->
   </joint>
   <link name="camera_rgb_frame" />

Commit message: ongoing : moving stick

File: basic_stick/urdf/moving_stick.xacro (robot description, xacro)
@@ -98,9 +98,10 @@
     <origin xyz="0 0 ${length1/2+length2/2}" rpy="0 0 -${pi/2}"/>
   </joint>
-  <joint name="tilt_joint" type="fixed">
+  <joint name="tilt_joint" type="revolute">
     <origin xyz="0.05 0 ${length2/2+0.02}" rpy="0 0.5 0" />
     <parent link="link_2" />
     <child link="camera_link" />
-    <!-- <axis xyz="0 1 0"/> -->
+    <limit lower="-1.5707" upper="1.5707" effort="10" velocity="100" />
+    <axis xyz="0 1 0"/>
   </joint>
   <link name="camera_rgb_frame" />

File: basic_stick/urdf/sensor_stick.xacro (robot description, xacro)
@@ -97,9 +97,9 @@
     <origin xyz="0 0 ${length1/2+length2/2}" rpy="0 0 -${pi/2}"/>
   </joint>
-  <joint name="tilt_joint" type="revolute">
+  <joint name="tilt_joint" type="fixed">
     <origin xyz="0.05 0 ${length2/2+0.02}" rpy="0 0.5 0" />
     <parent link="link_2" />
     <child link="camera_link" />
-    <axis xyz="0 1 0"/>
+    <!-- <axis xyz="0 1 0"/> -->
   </joint>
   <link name="camera_rgb_frame" />
