Commit message: fusion bot

File: fusionbot_description/urdf/fusionbot.urdf.xacro (robot description, xacro)
@@ -2,5 +2,5 @@
 <robot name="fusionbot" xmlns:xacro="http://www.ros.org/wiki/xacro">
   <xacro:include filename="$(find fusionbot_description)/urdf/materials.xacro" />
-  <xacro:include filename="$(find fusionbot_description)/urdf/fusionbot.gazebo" />
+  <!-- <xacro:include filename="$(find fusionbot_description)/urdf/fusionbot.gazebo" /> -->
   <link name='base_footprint' />
   <link name="base_link">
@@ -13,5 +13,5 @@
       <origin rpy="0 0 0" xyz="0 0 0" />
       <geometry>
-        <mesh filename="model://fusionbot/meshes/fusionbot/base_link.stl" scale="0.001 0.001 0.001" />
+        <mesh filename="$(find fusionbot_description)/meshes/base_link.stl" scale="0.001 0.001 0.001" />
       </geometry>
       <material name="silver" />
@@ -20,9 +20,9 @@
       <origin rpy="0 0 0" xyz="0 0 0" />
       <geometry>
-        <mesh filename="model://fusionbot/meshes/fusionbot/base_link.stl" scale="0.001 0.001 0.001" />
+        <mesh filename="$(find fusionbot_description)/meshes/base_link.stl" scale="0.001 0.001 0.001" />
       </geometry>
     </collision>
   </link>
-  <link name="right_wheel_1">
+  <link name="right_wheel">
     <inertial>
       <origin rpy="0 0 0" xyz="-5.790023100122029e-18 -0.012499999999999997 0.0" />
@@ -33,5 +33,5 @@
       <origin rpy="0 0 0" xyz="-0.0 0.1 -0.05" />
       <geometry>
-        <mesh filename="model://fusionbot/meshes/fusionbot/right_wheel_1.stl" scale="0.001 0.001 0.001" />
+        <mesh filename="$(find fusionbot_description)/meshes/right_wheel_1.stl" scale="0.001 0.001 0.001" />
       </geometry>
       <material name="silver" />
@@ -40,9 +40,9 @@
       <origin rpy="0 0 0" xyz="-0.0 0.1 -0.05" />
       <geometry>
-        <mesh filename="model://fusionbot/meshes/fusionbot/right_wheel_1.stl" scale="0.001 0.001 0.001" />
+        <mesh filename="$(find fusionbot_description)/meshes/right_wheel_1.stl" scale="0.001 0.001 0.001" />
       </geometry>
     </collision>
   </link>
-  <link name="left_wheel_1">
+  <link name="left_wheel">
     <inertial>
       <origin rpy="0 0 0" xyz="-5.790023100122029e-18 0.012499999999999997 0.0" />
@@ -53,5 +53,5 @@
       <origin rpy="0 0 0" xyz="-0.0 -0.1 -0.05" />
       <geometry>
-        <mesh filename="model://fusionbot/meshes/fusionbot/left_wheel_1.stl" scale="0.001 0.001 0.001" />
+        <mesh filename="$(find fusionbot_description)/meshes/left_wheel_1.stl" scale="0.001 0.001 0.001" />
       </geometry>
       <material name="silver" />
@@ -60,9 +60,9 @@
       <origin rpy="0 0 0" xyz="-0.0 -0.1 -0.05" />
       <geometry>
-        <mesh filename="model://fusionbot/meshes/fusionbot/left_wheel_1.stl" scale="0.001 0.001 0.001" />
+        <mesh filename="$(find fusionbot_description)/meshes/left_wheel_1.stl" scale="0.001 0.001 0.001" />
       </geometry>
     </collision>
   </link>
-  <link name="lidar_1">
+  <link name="lidar">
     <inertial>
       <origin rpy="0 0 0" xyz="0.0 0.0 0.012499999999999997" />
@@ -73,5 +73,5 @@
       <origin rpy="0 0 0" xyz="-0.05 -0.0 -0.11" />
       <geometry>
-        <mesh filename="model://fusionbot/meshes/fusionbot/lidar_1.stl" scale="0.001 0.001 0.001" />
+        <mesh filename="$(find fusionbot_description)/meshes/lidar_1.stl" scale="0.001 0.001 0.001" />
       </geometry>
       <material name="silver" />
@@ -80,5 +80,5 @@
       <origin rpy="0 0 0" xyz="-0.05 -0.0 -0.11" />
       <geometry>
-        <mesh filename="model://fusionbot/meshes/fusionbot/lidar_1.stl" scale="0.001 0.001 0.001" />
+        <mesh filename="$(find fusionbot_description)/meshes/lidar_1.stl" scale="0.001 0.001 0.001" />
       </geometry>
     </collision>
@@ -104,5 +104,5 @@
     <origin rpy="0 0 0" xyz="0.0 -0.1 0.05" />
     <parent link="base_link" />
-    <child link="right_wheel_1" />
+    <child link="right_wheel" />
     <axis xyz="0.0 1.0 0.0" />
   </joint>
@@ -110,5 +110,5 @@
     <origin rpy="0 0 0" xyz="0.0 0.1 0.05" />
     <parent link="base_link" />
-    <child link="left_wheel_1" />
+    <child link="left_wheel" />
     <axis xyz="0.0 1.0 0.0" />
   </joint>
@@ -128,5 +128,5 @@
     <origin rpy="0 0 0" xyz="0.05 0.0 0.11" />
     <parent link="base_link" />
-    <child link="lidar_1" />
+    <child link="lidar" />
   </joint>
 </robot>

File: fusionbot_description/urdf/fusionbot_description.urdf (robot description, URDF)
Before this commit: robot fusionbot, 7 links, 6 joints
Links:
- removed link left_wheel_1
- removed link lidar_1
- removed link right_wheel_1
- added link left_wheel, mass 0.1826050729899067; collision mesh filename=$(find fusionbot_description)/meshes/left_wheel_1.stl scale=0.001 0.001 0.001; visual mesh filename=$(find fusionbot_description)/meshes/left_wheel_1.stl scale=0.001 0.001 0.001
- added link lidar, mass 0.7552585088770711; collision mesh filename=$(find fusionbot_description)/meshes/lidar_1.stl scale=0.001 0.001 0.001; visual mesh filename=$(find fusionbot_description)/meshes/lidar_1.stl scale=0.001 0.001 0.001
- added link right_wheel, mass 0.1826050729899067; collision mesh filename=$(find fusionbot_description)/meshes/right_wheel_1.stl scale=0.001 0.001 0.001; visual mesh filename=$(find fusionbot_description)/meshes/right_wheel_1.stl scale=0.001 0.001 0.001
- link base_link: geometry collision mesh filename=$(find fusionbot_description)/meshes/base_link.stl scale=0.001 0.001 0.001; visual mesh filename=$(find fusionbot_description)/meshes/base_link.stl scale=0.001 0.001 0.001
Joints:
- joint left_wheel_joint: child left_wheel_1 -> left_wheel
- joint lidar_joint: child lidar_1 -> lidar
- joint right_wheel_joint: child right_wheel_1 -> right_wheel

File: fusionbot_description/urdf/materials.xacro (robot description, xacro)
@@ -16,3 +16,28 @@
     <color rgba="0 0 0.8 1"/>
   </material>
+  <gazebo reference="base_link">
+    <material>Gazebo/Silver</material>
+    <mu1>0.5</mu1>
+    <mu2>0.5</mu2>
+    <selfCollide>true</selfCollide>
+    <gravity>true</gravity>
+  </gazebo>
+  <gazebo reference="lidar">
+    <material>Gazebo/Blue</material>
+    <mu1>0.2</mu1>
+    <mu2>0.2</mu2>
+    <selfCollide>true</selfCollide>
+  </gazebo>
+  <gazebo reference="right_wheel">
+    <material>Gazebo/Black</material>
+    <mu1>100000.0</mu1>
+    <mu2>100000.0</mu2>
+    <selfCollide>true</selfCollide>
+  </gazebo>
+  <gazebo reference="left_wheel">
+    <material>Gazebo/Black</material>
+    <mu1>100000.0</mu1>
+    <mu2>100000.0</mu2>
+    <selfCollide>true</selfCollide>
+  </gazebo>
 </robot>
