Commit message: ongoing : bf lecture

File: fusionbot_description/urdf/fusionbot_description.urdf (robot description, URDF)
Before this commit: robot fusionbot, 7 links, 6 joints
Links:
- link base_link: geometry collision mesh filename=package://fusionbot_description/meshes/base_link.stl scale=0.001 0.001 0.001; visual mesh filename=package://fusionbot_description/meshes/base_link.stl scale=0.001 0.001 0.001
- link left_wheel: geometry collision mesh filename=package://fusionbot_description/meshes/left_wheel_1.stl scale=0.001 0.001 0.001; visual mesh filename=package://fusionbot_description/meshes/left_wheel_1.stl scale=0.001 0.001 0.001
- link lidar: geometry collision mesh filename=package://fusionbot_description/meshes/lidar_1.stl scale=0.001 0.001 0.001; visual mesh filename=package://fusionbot_description/meshes/lidar_1.stl scale=0.001 0.001 0.001
- link right_wheel: geometry collision mesh filename=package://fusionbot_description/meshes/right_wheel_1.stl scale=0.001 0.001 0.001; visual mesh filename=package://fusionbot_description/meshes/right_wheel_1.stl scale=0.001 0.001 0.001
