Commit message: Ongoing : lidar world laptop run

File: lidar_world/urdf/sensor_stick.urdf.xacro (robot description, xacro)
@@ -12,5 +12,5 @@
   <!--Import gazebo elements-->
   <!-- <xacro:include filename="$(find lidar_world)/urdf/sensor_stick.gazebo.xacro" /> -->
-  <!-- <xacro:include filename="$(find lidar_world)/urdf/sensor_stick_gpu.gazebo.xacro" /> -->
+  <xacro:include filename="$(find lidar_world)/urdf/sensor_stick_gpu.gazebo.xacro" />
   <!--Links-->
   <link name="world"/>
@@ -74,5 +74,5 @@
     <visual>
       <geometry>
-        <mesh filename="$(find velodyne_description)/meshes/VLP16_base_1.dae"/>
+        <mesh filename="$(find lidar_world)/meshes/VLP16_base_1.dae"/>
       </geometry>
     </visual>
@@ -93,5 +93,5 @@
       <origin xyz="0 0 -0.0377"/>
       <geometry>
-        <mesh filename="$(find velodyne_description)/meshes/VLP16_scan.dae"/>
+        <mesh filename="$(find lidar_world)/meshes/VLP16_scan.dae"/>
       </geometry>
     </visual>
@@ -106,5 +106,5 @@
       <origin xyz="0 0 -0.0377"/>
       <geometry>
-        <mesh filename="$(find velodyne_description)/meshes/VLP16_base_2.dae"/>
+        <mesh filename="$(find lidar_world)/meshes/VLP16_base_2.dae"/>
       </geometry>
     </visual>
